File: Board/board.brd (EAGLE design)
At the start: 50 x 50 mm, 31 parts, among them IC1 MCP2300X/SO, IC2 LM1117, U1 ADS1015

Commit message: Use cheaper ADC and add LEDs on spare GPIO
Parts:
- removed U1: ADS1015, SparkFun-AnalogIC:MSOP10
- added LED4, LED5, LED6: (no value), microbuilder:CHIPLED_0805
- added R1, R6, R9: 70, resistor:R0603
- added U2: MAX11607EUA+T, MAX11607:21-0036K
Connections:
- new net N$11: LED6.C, R9.1
- new net N$7: LED4.C, R1.1
- new net N$9: LED5.C, R6.1
- net +3V3: now also GP3.P$1, GP4.P$1, LED4.A, LED5.A, LED6.A, U2.4, U2.8; no longer U1.8
- net GND: now also R1.2, U2.7; no longer GP3.P$1, GP4.P$1, U1.1, U1.3
- net GP6: now also IC1.17, R6.2; no longer IC1.16
- net GP7: now also IC1.16, R9.2; no longer IC1.17
- net I2C_SCL: now also U2.5; no longer U1.10
- net I2C_SDA: now also U2.6; no longer U1.9
- net N$3: now also U2.3; no longer U1.6
- net N$4: now also U2.2; no longer U1.5
- net N$5: now also U2.1; no longer U1.4
Routing:
- net GND: track 279.2 -> 237.1 mm
- net +3V3: track 181.3 -> 207.4 mm
- net N$7: track 0.00 -> 5.56 mm
- net I2C_SDA: track 62.6 -> 57.8 mm
- net N$2: track 21.0 -> 25.2 mm, vias 0 -> 1
- net N$9: track 0.00 -> 3.84 mm
- net GP6: track 39.9 -> 43.7 mm
- net N$11: track 0.00 -> 3.59 mm
- net I2C_SCL: track 58.6 -> 55.3 mm
- net N$3: track 8.03 -> 10.7 mm
- net N$4: track 2.21 -> 4.06 mm
- net N$5: track 11.8 -> 13.6 mm
- net VCC: track 10.8 -> 11.7 mm
Other:
- board text added: "Arbitos kleinpa.net REVA"
- board text removed: "Switch kleinpa.net REVA"

Commit message: Finish routing PCB
Parts:
- removed D4: (no value), diode:DO214AC
- removed DC-IN: POWER_JACKPTH, SparkFun-Connectors:POWER_JACK_PTH
- removed ESP-01: ESP01, esp8266modules-pk:ESP01
- removed GP3, GP4: 02-JST, con-jst-xh:B2B-XH
- removed IC1: MCP2300X/SO, adafruit:SO18W
- removed JP2: FTDI_DEVICE, SparkFun-Connectors:FTDI_DEVICE_SIDE
- removed LED5, LED6: (no value), microbuilder:CHIPLED_0805
- removed U2: MAX11607EUA+T, MAX11607:21-0036K
- added C1: 47pF, rcl:C0603
- added C5: 10nF, rcl:C0603
- added D1, D2, D3: (no value), diode:DO214AC
- added L1: (no value), SparkFun-Passives:0805
- added T1, T2: (no value), transistor:SOT23-BEC
- added U1: FTS31XS-U, SparkFun-DigitalIC:SSOP20_L
- added USB: USB-RECEPTABLE, daspilker:FCI-10103594-0001LF
- added X1: (no value), adafruit:ESP-12
- C4: value .1uF -> 47pF; device SparkFun-Passives:0603-CAP -> rcl:C0603
- R6: value 70 -> 27
- R7: value 10k -> 27
- R8: value 10k -> 12k
- R9: value 70 -> 12k
- moved R9 28.4 mm to (17.1, 34.9), flipped to the bottom, turned to 0 degrees
- moved R6 25.6 mm to (17.8, 22.2), flipped to the bottom, turned to 90 degrees
- moved R4 23.4 mm to (41.3, 19.7), turned to 270 degrees
- moved R7 22.5 mm to (19.7, 22.2), turned to 90 degrees
- moved R8 20.5 mm to (17.1, 32.4), turned to 180 degrees
- moved C4 17.8 mm to (21.6, 22.2), turned to 270 degrees
- moved H1 10.2 mm to (47.0, 13.2)
- moved C2 4.26 mm to (38.1, 11.4)
- moved C3 4.26 mm to (33.7, 11.4)
- moved IC2 2.29 mm to (31.8, 18.4)
- moved R1 1.27 mm to (43.2, 19.7), flipped to the bottom, turned to 90 degrees
- moved LED4 0.74 mm to (47.0, 18.7)
Connections:
- removed net GP0: IC1.10, S1.1, S1.2
- removed net GP1: IC1.11, LED1.K
- removed net GP2: IC1.12, S2.1, S2.2
- removed net GP3: IC1.13, LED2.K
- removed net GP4: IC1.14, S3.1, S3.2
- removed net GP5: IC1.15, LED3.K
- removed net GP6: GP3.P$2, IC1.17, R6.2
- removed net GP7: GP4.P$2, IC1.16, R9.2
- removed net I2C_SCL: ESP-01.GPIO2, IC1.1, R8.1, U2.5
- removed net I2C_SDA: D4.A, ESP-01.GPIO0, IC1.2, R7.1, U2.6
- removed net VCC: C2.+, DC-IN.PWR, IC2.3
- new net ADC: D1.C, D2.C, D3.C, X1.2
- new net GPIO0: S2.1, S2.2, T2.C, X1.12
- new net GPIO12: LED1.K, X1.6
- new net GPIO13: S1.1, S1.2, X1.7
- new net GPIO14: LED2.K, X1.5
- new net GPIO15: VR2.P$3, X1.10
- new net GPIO16: LED3.K, X1.4
- new net GPIO2: S3.1, S3.2, X1.11
- new net GPIO4: VR0.P$3, X1.14
- new net GPIO5: VR1.P$3, X1.13
- new net N$12: D3.A, VR2.P$2
- new net N$13: C1.2, R6.1, USB.2
- new net N$14: R8.1, T2.E, U1.1
- new net N$15: R9.1, T1.E, U1.2
- new net N$16: R8.2, T1.B
- new net N$17: R9.2, T2.B
- new net N$19: U1.13, U1.14, U1.3
- new net N$20: C2.+, IC2.3, L1.1, U1.15
- net +3V3: now also R1.1, X1.8; no longer ESP-01.VCC, GP3.P$1, GP4.P$1, IC1.18, IC1.6, LED4.A, LED5.A, LED6.A, R7.2, R8.2, U2.4, U2.8, VR0.P$3, VR1.P$3, VR2.P$3
- net GND: now also C1.1, C4.1, C5.1, LED4.C, U1.16, U1.6, USB.5, X1.9; no longer DC-IN.GND, DC-IN.GNDBREAK, ESP-01.GND, IC1.3, IC1.4, IC1.5, IC1.9, JP2.P$6, R1.2, U2.7
- net N$1: now also X1.3; no longer ESP-01.CH_PD
- net N$11: now also D2.A, VR1.P$2; no longer LED6.C, R9.1
- net N$2: now also R7.1, USB.3; no longer D4.C, JP2.P$1
- net N$3: now also R7.2, U1.11; no longer U2.3, VR2.P$2
- net N$4: now also LED4.A, R1.2; no longer U2.2, VR1.P$2
- net N$5: now also D1.A; no longer U2.1
- net N$7: now also C5.2, L1.2, USB.1; no longer LED4.C, R1.1
- net N$9: now also R6.2, U1.12; no longer LED5.C, R6.1
- net RST: now also T1.C, X1.1; no longer C4.1, ESP-01.RST
- net RXI: now also U1.20, X1.15; no longer ESP-01.RX, JP2.P$3
- net TXO: now also U1.4, X1.16; no longer ESP-01.TX, JP2.P$2
Routing:
- net +3V3: track 207.4 -> 103.2 mm, vias 4 -> 6
- net ADC: track 0.00 -> 83.4 mm, vias 0 -> 2
- net GPIO16: track 0.00 -> 68.9 mm, vias 0 -> 1
- net GPIO0: track 0.00 -> 62.9 mm
- net I2C_SDA: track 57.8 -> 0.00 mm, vias 2 -> 0
- net I2C_SCL: track 55.3 -> 0.00 mm, vias 2 -> 0
- net GPIO14: track 0.00 -> 55.2 mm, vias 0 -> 1
- net GP7: track 45.1 -> 0.00 mm, vias 1 -> 0
- net GP6: track 43.7 -> 0.00 mm, vias 1 -> 0
- net GPIO13: track 0.00 -> 42.5 mm
- net GPIO12: track 0.00 -> 41.9 mm
- net N$13: track 0.00 -> 39.4 mm, vias 0 -> 2
- net GPIO2: track 0.00 -> 36.8 mm
- net RXI: track 8.11 -> 40.9 mm
- net N$20: track 0.00 -> 31.7 mm, vias 0 -> 2
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- added copper zone on layer 1, net GND
- added copper zone on layer 16, net GND
Other:
- board text added: "C:/Users/klein/Projects/logo/logo.bmp"
- board text added: "POWER"
